Commit message: fix(unitree): gate trotting from nominal stance

File: src/unitree_guide/unitree_ros/robots/a1_description/xacro/leg.xacro (robot description, xacro)
@@ -136,12 +136,4 @@
             <child link="${name}_foot"/>
         </joint>
-        <joint name="${name}_foot_joint_get_position" type="revolute">
-            <origin rpy="0 0 0" xyz="0 0 ${-(calf_length)}"/>
-            <parent link="${name}_calf"/>
-            <child link="${name}_foot"/>
-            <axis xyz="0 1 0"/>
-            <dynamics damping="${damping}" friction="${friction}"/>
-            <limit effort="0" velocity="0" lower="0" upper="0"/>
-        </joint>
         <link name="${name}_foot">
             <visual>
